File: ESPHome_LED-Dimmer-V1.0.0.kicad_pcb (KiCad board)
At the start: 2 copper layers, 50 x 40 mm, 15 parts, among them J2 Screw_Terminal_01x04, Q1 IRF7842PbF, U1 ESP32-C3_SUPERMINI, U2 BuckConverter_5V/3A

Commit message: Final version 1.0.0 (for PCB production)
Parts:
- removed Logo3: http://fablabwinti.ch, CPs_Footprints:QR_FabLab-Winti
- added GitHub-Link1: https://yurl.ch?r=LedDim, CPs_Footprints:QR_GitHub-LedDim, B.Cu at (95.0, 78.4)
- J1: renamed from J2; value Screw_Terminal_01x04 -> Screw_Terminal_1x4, P3.81mm
- LED1: value EL 15-21/G6C-FP1Q1L/2T -> 15-21/G6C-FP1Q1L/2T
- moved R3 0.89 mm to (125.5, 78.0)
- moved R2 0.25 mm to (116.2, 83.1)
- moved H3 0.20 mm to (131.1, 96.4)
- moved H2 0.13 mm to (86.2, 96.4)
- renumbered Q1 to FET1, Logo1 to KiCad-Logo1, Logo2 to OpenHardware-Logo1
Connections:
- J1 pad 1: /12V -> /GND
- J1 pad 2: /GND -> /12V
Routing:
- net Net-(LED1-K): track 3.59 -> 5.37 mm
- net /12V: track 27.2 -> 28.2 mm
Other:
- board size 50 x 40 mm -> 49.9 x 39.9 mm
- board text added: "V1.0.0 (06.03.2025)"
- board text removed: "V1.0.0 (28.02.2025)"
