File: ESPHome_LED-Dimmer-V1.0.0.kicad_sch (KiCad schematic)
At the start: 15 parts, among them J2 Screw_Terminal_01x04, Q1 IRF7842PbF, U1 ESP32-C3_SUPERMINI, U2 BuckConverter_5V/3A

Commit message: Final version 1.0.0 (for PCB production)
Parts:
- removed Logo3: http://fablabwinti.ch, CPs_Footprints:QR_FabLab-Winti, symbol A_SymbolLibrary:MountingHole
- added GitHub-Link1: https://yurl.ch?r=LedDim, CPs_Footprints:QR_GitHub-LedDim, symbol ESPHome_LED-Diimmer_Symbols:MountingHole
- FET1: renamed from Q1; symbol Transistor_FET:IRF740 -> ESPHome_LED-Diimmer_Symbols:IRF740
- H1, H2, H3, H4: symbol A_SymbolLibrary:MountingHole -> ESPHome_LED-Diimmer_Symbols:MountingHole
- J1: renamed from J2; value Screw_Terminal_01x04 -> Screw_Terminal_1x4, P3.5mm; symbol Connector:Screw_Terminal_01x04 -> ESPHome_LED-Diimmer_Symbols:Screw_Terminal_01x04
- KiCad-Logo1: renamed from Logo1; symbol A_SymbolLibrary:MountingHole -> ESPHome_LED-Diimmer_Symbols:MountingHole
- LED1: value EL 15-21/G6C-FP1Q1L/2T -> 15-21/G6C-FP1Q1L/2T; symbol LED:IR26-21C_L110_TR8 -> ESPHome_LED-Diimmer_Symbols:IR26-21C_L110_TR8
- OpenHardware-Logo1: renamed from Logo2; symbol A_SymbolLibrary:MountingHole -> ESPHome_LED-Diimmer_Symbols:MountingHole
- R1, R2, R3: symbol A_SymbolLibrary:R -> ESPHome_LED-Diimmer_Symbols:R
- U1: symbol A_SymbolLibrary:ESP32-C3_SUPERMINI -> ESPHome_LED-Diimmer_Symbols:ESP32-C3_SUPERMINI
- U2: symbol A_SymbolLibrary:module_BuckConverter_Mini560 -> ESPHome_LED-Diimmer_Symbols:module_BuckConverter_Mini560
Connections:
- net 12V: now also J1.2 (Pin_2); no longer J1.1 (Pin_1)
- net GND: now also J1.1 (Pin_1); no longer J1.2 (Pin_2)
